File: PCB_Parts/main_board/main.kicad_sch (KiCad schematic)
At the start: 4 parts, among them J1 Conn_01x20_Socket, J2 Conn_01x20_Socket, J3 Conn_01x20_Socket, J4 Conn_01x20_Socket

Commit message: a
Connections:
- net Pico_AGND: now also J4.13 (Pin_13); no longer J4.14 (Pin_14)
- net Pico_RUN: now also J4.11 (Pin_11); no longer J4.12 (Pin_12)
- net 2W_VBUS: now reaches J2.1 (Pin_1)
- net VBAT_ADC: now reaches J2.11 (Pin_11)
- net 2W_RUN: now reaches J2.12 (Pin_12)
- net 2W_AGND: now reaches J2.14 (Pin_14)
- net 2W_AGND: now also J1.13 (Pin_13), J1.18 (Pin_18), J1.3 (Pin_3), J1.8 (Pin_8), J2.18 (Pin_18), J2.3 (Pin_3), J2.8 (Pin_8)
- net 2W_VSYS: now reaches J2.2 (Pin_2)
- net 2W_EN: now reaches J2.4 (Pin_4)
- net 2W_3V3_OUT: now reaches J2.5 (Pin_5)
- net 2W_ADC_VREF: now reaches J2.6 (Pin_6)
- net M1_PH: now reaches J3.1 (Pin_1)
- net M4_EN: now reaches J3.10 (Pin_10)
- net Pico_UART_TX: now reaches J3.11 (Pin_11)
- net Pico_UART_RX: now reaches J3.12 (Pin_12)
- net DRV_nSLEEP: now reaches J3.14 (Pin_14)
- net DRV_nFAULT: now reaches J3.15 (Pin_15)
- net DRIBBLER_PWM: now reaches J3.16 (Pin_16)
- net DRIBBLER_DIR: now reaches J3.17 (Pin_17)
- net DRIBBLER_ENABLE: now reaches J3.19 (Pin_19)
- net M1_EN: now reaches J3.2 (Pin_2)
- net KICK: now reaches J3.20 (Pin_20)
- net M2_PH: now reaches J3.4 (Pin_4)
- net M2_EN: now reaches J3.5 (Pin_5)
- net M3_PH: now reaches J3.6 (Pin_6)
- net M3_EN: now reaches J3.7 (Pin_7)
- net M4_PH: now reaches J3.9 (Pin_9)
- net REAR_ECHO: now reaches J4.10 (Pin_10)
- net RIGHT_TRIG: now reaches J4.15 (Pin_15)
- net LEFT_ECHO: now reaches J4.16 (Pin_16)
- net LEFT_TRIG: now reaches J4.17 (Pin_17)
- net FRONT_ECHO: now reaches J4.19 (Pin_19)
- net FRONT_TRIG: now reaches J4.20 (Pin_20)
- net 2W_I2C_SDA: now reaches J1.1 (Pin_1)
- net IR_EN: now reaches J1.10 (Pin_10)
- net 2W_UART_TX: now reaches J1.11 (Pin_11)
- net 2W_UART_RX: now reaches J1.12 (Pin_12)
- net IR_OUT_A: now reaches J1.14 (Pin_14)
- net IR_OUT_B: now reaches J1.15 (Pin_15)
- net LED1: now reaches J1.17 (Pin_17)
- net LED2: now reaches J1.19 (Pin_19)
- net 2W_I2C_SCL: now reaches J1.2 (Pin_2)
- net Buzzer: now reaches J1.20 (Pin_20)
- net BNO085_H_INTN: now reaches J1.4 (Pin_4)
- net BNO085_NRST: now reaches J1.5 (Pin_5)
- net IR_S0: now reaches J1.6 (Pin_6)
- net IR_S1: now reaches J1.7 (Pin_7)
- net IR_S2: now reaches J1.9 (Pin_9)
- net Pico_3V3 renamed Pico_3V3_OUT
- new net REAR_TRIG: J4.12 (Pin_12)
- new net RIGHT_ECHO: J4.14 (Pin_14)
Other:
- note added: "BNO085"
- note added: "DRIBBLER"
- note added: "IR"
- note added: "KICK"
- note added: "MOTOR/I2C"
- note added: "SUPERSONIC"
- note added: "UART"
- moved on the sheet: J1, J2

Commit message: BBB
Parts:
- added C1, C11, C16, C21: 22nF, Capacitor_SMD:C_0603_1608Metric, symbol Device:C
- added C10, C13, C15, C18, C20, C3, C5, C8: 100nF, Capacitor_SMD:C_0603_1608Metric, symbol Device:C
- added C12, C17, C4, C7: 10nF, Capacitor_SMD:C_0603_1608Metric, symbol Device:C
- added C14, C19, C6, C9: 470nF, Capacitor_SMD:C_0603_1608Metric, symbol Device:C
- added C2: 3.3nF, Capacitor_SMD:C_0603_1608Metric, symbol Device:C
- added J5: Conn_01x02, Connector_AMASS:AMASS_XT30PW-M_1x02_P2.50mm_Horizontal, symbol Connector_Generic:Conn_01x02
- added L1, L2: 2.2uH, Inductor_SMD:L_Coilcraft_XxL4020, symbol Device:L
- added R1, R10, R12, R2, R4, R6, R7, R9: 2.2kΩ, Resistor_SMD:R_0603_1608Metric, symbol Device:R
- added R11, R3, R5, R8: 22kΩ, Resistor_SMD:R_0603_1608Metric, symbol Device:R
- added U1, U2, U3, U4: DRV8874PWPR, PWP0016J_N, symbol KiCADv6:DRV8874PWPR
- added U121: TPS62133, Package_DFN_QFN:VQFN-16-1EP_3x3mm_P0.5mm_EP1.68x1.68mm_ThermalVias, symbol Regulator_Switching:TPS62133
- added U1211: TPS62162DSG, Package_SON:Texas_DSG0008A_WSON-8-1EP_2x2mm_P0.5mm_EP0.9x1.6mm_ThermalVias, symbol Regulator_Switching:TPS62162DSG
- added U5, U6: CD74HC4051PWR, PW16, symbol 2026-10-01_06-26-45:CD74HC4051PWR
- added U7: ADS1015IDGS, Package_SO:TSSOP-10_3x3mm_P0.5mm, symbol Analog_ADC:ADS1015IDGS
- J2, J4: footprint Connector_PinHeader_2.54mm:PinHeader_1x20_P2.54mm_Vertical -> Connector_PinSocket_2.54mm:PinSocket_1x20_P2.54mm_Vertical
Connections:
- net 2W_I2C_SCL: now also U7.10 (SCL)
- net 2W_I2C_SDA: now also U7.9 (SDA)
- net DRV_nFAULT: now also U1.4 (FAULT_N), U2.4 (FAULT_N), U3.4 (FAULT_N), U4.4 (FAULT_N)
- net DRV_nSLEEP: now also U1.3 (SLEEP_N), U2.3 (SLEEP_N), U3.3 (SLEEP_N), U4.3 (SLEEP_N)
- net IR_EN: now also U5.6 (*E), U6.6 (*E)
- net IR_OUT_A: now also U5.3 (A)
- net IR_OUT_B: now also U6.3 (A)
- net IR_S0: now also U5.11 (S0), U6.11 (S0)
- net IR_S1: now also U5.10 (S1), U6.10 (S1)
- net IR_S2: now also U5.9 (S2), U6.9 (S2)
- net M1_EN: now also U1.1 (EN_IN1)
- net M1_PH: now also U1.2 (PH_IN2)
- net M2_EN: now also U2.1 (EN_IN1)
- net M2_PH: now also U2.2 (PH_IN2)
- net M3_EN: now also U3.1 (EN_IN1)
- net M3_PH: now also U3.2 (PH_IN2)
- net M4_EN: now also U4.1 (EN_IN1)
- net M4_PH: now also U4.2 (PH_IN2)
- new net: R7.2, R8.1, U3.5 (VREF)
- new net: C3.2, U1.12 (VCP)
- new net: C1.1, U1.13 (CPH)
- new net: C1.2, U1.14 (CPL)
- new net: R2.2, R3.1, U1.5 (VREF)
- new net: C4.2, R1.2, U1.6 (IPROPI)
- new net: R4.2, R5.1, U2.5 (VREF)
- new net: C10.2, U2.12 (VCP)
- new net: C11.1, U2.13 (CPH)
- new net: C11.2, U2.14 (CPL)
- new net: C7.2, R6.2, U2.6 (IPROPI)
- new net: L1.1, U121.1 (SW), U121.2 (SW), U121.3 (SW)
- new net: C2.2, U121.9 (SS/TR)
- new net: C17.2, R12.2, U4.6 (IPROPI)
- new net: L2.1, U1211.7 (SW)
- new net: C15.2, U3.12 (VCP)
- new net: C16.1, U3.13 (CPH)
- new net: C16.2, U3.14 (CPL)
- new net: C12.2, R9.2, U3.6 (IPROPI)
- new net: C20.2, U4.12 (VCP)
- new net: R10.2, R11.1, U4.5 (VREF)
- new net: C21.1, U4.13 (CPH)
- new net: C21.2, U4.14 (CPL)
- new net 3V3_AUX: L2.2, R10.1, R2.1, R4.1, R7.1, U1211.6 (VOS), U5.16 (VCC), U6.16 (VCC), U7.8 (VDD)
- new net 5V: L1.2, U121.14 (VOS), U1211.2 (VIN), U1211.3 (EN)
- new net GND: C12.1, C13.1, C14.1, C17.1, C18.1, C19.1, C2.1, C4.1, C5.1, C6.1, C7.1, C8.1, C9.1, J5.1 (Pin_1), R1.1, R11.2, R12.1, R3.2, R5.2, R6.1, R8.2, R9.1, U1.15 (GND), U1.16 (PMODE), U1.17 (PAD), U1.7 (IMODE), U1.9 (PGND), U121.15 (GND), U121.16 (GND), U121.17 (GND), U121.5 (FB), U121.6 (GND), U121.7 (FSW), U121.8 (DEF), U1211.1 (PGND), U1211.4 (AGND), U1211.5 (FB), U1211.9 (PAD), U2.15 (GND), U2.16 (PMODE), U2.17 (PAD), U2.7 (IMODE), U2.9 (PGND), U3.15 (GND), U3.16 (PMODE), U3.17 (PAD), U3.7 (IMODE), U3.9 (PGND), U4.15 (GND), U4.16 (PMODE), U4.17 (PAD), U4.7 (IMODE), U4.9 (PGND), U5.7 (VEE), U5.8 (GND), U6.7 (VEE), U6.8 (GND), U7.1 (ADDR), U7.3 (GND)
- new net IR_LING_CH1: U5.13 (A0)
- new net IR_LING_CH10: U6.14 (A1)
- new net IR_LING_CH11: U6.15 (A2)
- new net IR_LING_CH12: U6.12 (A3)
- new net IR_LING_CH2: U5.14 (A1)
- new net IR_LING_CH3: U5.15 (A2)
- new net IR_LING_CH4: U5.12 (A3)
- new net IR_LING_CH9: U6.13 (A0)
- new net IR_OUT_CH13: U6.1 (A4)
- new net IR_OUT_CH14: U6.5 (A5)
- new net IR_OUT_CH15: U6.2 (A6)
- new net IR_OUT_CH16: U6.4 (A7)
- new net IR_OUT_CH5: U5.1 (A4)
- new net IR_OUT_CH6: U5.5 (A5)
- new net IR_OUT_CH7: U5.2 (A6)
- new net IR_OUT_CH8: U5.4 (A7)
- new net LINE_FRONT: U7.4 (AIN0)
- new net LINE_LEFT: U7.5 (AIN1)
- new net LINE_REAR: U7.7 (AIN3)
- new net LINE_RIGHT: U7.6 (AIN2)
- new net MOTOR1_OUT1: U1.8 (OUT1)
- new net MOTOR1_OUT2: U1.10 (OUT2)
- new net MOTOR2_OUT1: U2.8 (OUT1)
- new net MOTOR2_OUT2: U2.10 (OUT2)
- new net MOTOR3_OUT1: U3.8 (OUT1), U4.8 (OUT1)
- new net MOTOR3_OUT2: U3.10 (OUT2), U4.10 (OUT2)
- new net VBAT_FUSED: C10.1, C13.2, C14.2, C15.1, C18.2, C19.2, C20.1, C3.1, C5.2, C6.2, C8.2, C9.2, U1.11 (VM), U121.10 (VIN), U121.11 (VIN), U121.12 (VIN), U121.13 (EN), U2.11 (VM), U3.11 (VM), U4.11 (VM)
Other:
- company: (none) -> w(ﾟДﾟ)w
- title: (none) -> ヾ(•ω•`)o
- moved on the sheet: J1, J2, J3, J4

Commit message: aa
Parts:
- added C22: C_Polarized, Capacitor_SMD:CP_Elec_10x10.5, symbol Device:C_Polarized
- added D1, D2: D_Schottky, Diode_SMD:D_SMA, symbol Device:D_Schottky
- added F1: 20A, Fuse:Fuse_1206_3216Metric, symbol Device:Fuse
- added J10: Conn_01x05, Connector_PinSocket_2.54mm:PinSocket_1x05_P2.54mm_Vertical, symbol Connector_Generic:Conn_01x05
- added J11, J12, J13, J14: Conn_01x04, Connector_JST:JST_PH_B4B-PH-K_1x04_P2.00mm_Vertical, symbol Connector_Generic:Conn_01x04
- added J15, J16: Conn_01x08, Connector_JST:JST_PH_B8B-PH-K_1x08_P2.00mm_Vertical, symbol Connector_Generic:Conn_01x08
- added J17, J18, J19, J20: Conn_01x03, Connector_JST:JST_PH_S3B-PH-K_1x03_P2.00mm_Horizontal, symbol Connector_Generic:Conn_01x03
- added J21, J22, J6, J7, J8, J9: Screw_Terminal_01x02, TerminalBlock_Phoenix:TerminalBlock_Phoenix_MKDS-1,5-2-5.08_1x02_P5.08mm_Horizontal, symbol Connector:Screw_Terminal_01x02
- added R13, R16: 100Ω, Resistor_SMD:R_0603_1608Metric, symbol Device:R
- added R14, R15: 100kΩ, Resistor_SMD:R_0603_1608Metric, symbol Device:R
- added U8, U9: IRLML6344TRPBF, IRLML6344TRPBF_INF, symbol 2026-10-05_00-38-08:IRLML6344TRPBF
Connections:
- net 2W_I2C_SCL: now also J10.5 (Pin_5)
- net 2W_I2C_SDA: now also J10.4 (Pin_4)
- net 3V3_AUX: now also J10.1 (Pin_1), J11.1 (Pin_1), J12.1 (Pin_1), J13.1 (Pin_1), J14.1 (Pin_1), J17.2 (Pin_2), J18.2 (Pin_2), J19.2 (Pin_2), J20.2 (Pin_2)
- net BNO085_H_INTN: now also J10.3 (Pin_3)
- net DRIBBLER_PWM: now also R13.2
- net FRONT_ECHO: now also J11.3 (Pin_3)
- net FRONT_TRIG: now also J11.2 (Pin_2)
- net GND: now also C12.2, C22.2, J10.2 (Pin_2), J11.4 (Pin_4), J12.4 (Pin_4), J13.4 (Pin_4), J14.4 (Pin_4), J17.1 (Pin_1), J18.1 (Pin_1), J19.1 (Pin_1), J20.1 (Pin_1), R14.2, R15.2, U8.2 (S), U9.2 (S); no longer C12.1
- net IR_LING_CH1: now also J15.1 (Pin_1)
- net IR_LING_CH10: now also J16.2 (Pin_2)
- net IR_LING_CH11: now also J16.3 (Pin_3)
- net IR_LING_CH12: now also J16.4 (Pin_4)
- net IR_LING_CH2: now also J15.2 (Pin_2)
- net IR_LING_CH3: now also J15.3 (Pin_3)
- net IR_LING_CH4: now also J15.4 (Pin_4)
- net IR_LING_CH9: now also J16.1 (Pin_1)
- net KICK: now also R16.2
- net LEFT_ECHO: now also J12.3 (Pin_3)
- net LEFT_TRIG: now also J12.2 (Pin_2)
- net LINE_FRONT: now also J17.3 (Pin_3)
- net LINE_LEFT: now also J18.3 (Pin_3)
- net LINE_REAR: now also J20.3 (Pin_3)
- net LINE_RIGHT: now also J19.3 (Pin_3)
- net MOTOR1_OUT1: now also J6.1 (Pin_1)
- net MOTOR1_OUT2: now also J6.2 (Pin_2)
- net MOTOR2_OUT1: now also J7.1 (Pin_1)
- net MOTOR2_OUT2: now also J7.2 (Pin_2)
- net MOTOR3_OUT1: now also J8.1 (Pin_1); no longer U4.8 (OUT1)
- net MOTOR3_OUT2: now also J8.2 (Pin_2); no longer U4.10 (OUT2)
- net REAR_ECHO: now also J14.3 (Pin_3)
- net REAR_TRIG: now also J14.2 (Pin_2)
- net RIGHT_ECHO: now also J13.3 (Pin_3)
- net RIGHT_TRIG: now also J13.2 (Pin_2)
- net VBAT_FUSED: now also C22.1, D1.1 (K), D2.1 (K), F1.2, J21.1 (Pin_1), J22.1 (Pin_1)
- net at J5.2 (Pin_2): now also F1.1
- net at R9.2, U3.6 (IPROPI): now also C12.1; no longer C12.2
- net IR_OUT_CH13 renamed IR_LING_CH13
- net IR_LING_CH13: now also J16.5 (Pin_5)
- net IR_OUT_CH14 renamed IR_LING_CH14
- net IR_LING_CH14: now also J16.6 (Pin_6)
- net IR_OUT_CH15 renamed IR_LING_CH15
- net IR_LING_CH15: now also J16.7 (Pin_7)
- net IR_OUT_CH16 renamed IR_LING_CH16
- net IR_LING_CH16: now also J16.8 (Pin_8)
- net IR_OUT_CH5 renamed IR_LING_CH5
- net IR_LING_CH5: now also J15.5 (Pin_5)
- net IR_OUT_CH6 renamed IR_LING_CH6
- net IR_LING_CH6: now also J15.6 (Pin_6)
- net IR_OUT_CH7 renamed IR_LING_CH7
- net IR_LING_CH7: now also J15.7 (Pin_7)
- net IR_OUT_CH8 renamed IR_LING_CH8
- net IR_LING_CH8: now also J15.8 (Pin_8)
- new net: R13.1, R14.1, U8.1 (G)
- new net: R15.1, R16.1, U9.1 (G)
- new net DRIB_MOTOR_SW: D1.2 (A), J21.2 (Pin_2), U8.3 (D)
- new net KICK_SW: D2.2 (A), J22.2 (Pin_2), U9.3 (D)
- new net MOTOR4_OUT1: J9.1 (Pin_1), U4.8 (OUT1)
- new net MOTOR4_OUT2: J9.2 (Pin_2), U4.10 (OUT2)
Other:
- note added: "ADS1015(LINE)"
- note added: "BNO085(Conn)"
- note added: "Battery(Conn)"
- note added: "CD74HC4051(IR)"
- note added: "DRV8874"
- note added: "IR Ring(Conn)"
- note added: "Line(Conn)"
- note added: "Motor(Conn)"
- note added: "SuperSonic(Conn)"
- note added: "TPS62133(5V)"
- note added: "TPS62162(3V3)"
- moved on the sheet: C1, C10, C11, C12, C13, C14, C15, C16, C17, C18, C19, C2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

Commit message: j
Parts:
- removed J16: Conn_01x08, Connector_JST:JST_PH_B8B-PH-K_1x08_P2.00mm_Vertical, symbol Connector_Generic:Conn_01x08
- removed U5, U6: CD74HC4051PWR, PW16, symbol 2026-10-01_06-26-45:CD74HC4051PWR
- added C23: 1000uF, Capacitor_SMD:CP_Elec_10x10.5, symbol Device:C_Polarized
- added C24: 100nF, Capacitor_SMD:C_0603_1608Metric, symbol Device:C
- added R17: 10kΩ, Resistor_SMD:R_0603_1608Metric, symbol Device:R
- added R18: 2.7kΩ, Resistor_SMD:R_0603_1608Metric, symbol Device:R
- added TP1, TP2, TP3, TP4, TP5, TP6, TP7, TP8: TestPoint, TestPoint:TestPoint_Plated_Hole_D2.0mm, symbol Connector:TestPoint
- C22: value C_Polarized -> 1000uF
Connections:
- net 2W_VSYS is gone; now on net 5V: J2.2 (Pin_2)
- net IR_LING_CH1 is gone; now on net 3V3_AUX: J15.1 (Pin_1)
- net IR_LING_CH2 is gone; now on net GND: J15.2 (Pin_2)
- net IR_LING_CH3 is gone; now on net IR_S0: J15.3 (Pin_3)
- net IR_LING_CH4 is gone; now on net IR_S1: J15.4 (Pin_4)
- net IR_LING_CH5 is gone; now on net IR_S2: J15.5 (Pin_5)
- net IR_LING_CH6 is gone; now on net IR_EN: J15.6 (Pin_6)
- net IR_LING_CH7 is gone; now on net IR_OUT_A: J15.7 (Pin_7)
- net IR_LING_CH8 is gone; now on net IR_OUT_B: J15.8 (Pin_8)
- net Pico_UART_RX is gone; now on net 2W_UART_TX: J3.12 (Pin_12)
- net Pico_UART_TX is gone; now on net 2W_UART_RX: J3.11 (Pin_11)
- net Pico_VSYS is gone; now on net 5V: J4.2 (Pin_2)
- net 3V3_AUX: now also TP3.1
- net 5V: now also TP2.1
- net DRIB_MOTOR_SW: now also TP5.1
- net DRV_nFAULT: now also TP6.1
- net GND: now also C23.2, R18.1, TP7.1
- net KICK_SW: now also TP4.1
- net VBAT_ADC: now also C24.2, R17.1, R18.2, TP8.1
- net VBAT_FUSED: now also R17.2, TP1.1
- net at F1.1, J5.2 (Pin_2): now also C23.1
Other:
- note added: "BatADC"
- note added: "KICKER"
- note removed: "CD74HC4051(IR)"
- moved on the sheet: C1, C10, C11, C12, C13, C14, C15, C16, C17, C18, C19, C2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

Commit message: g
Parts:
- added D3, D4, D5, D6: LED, LED_SMD:LED_1206_3216Metric, symbol Device:LED
- added J23: Conn_01x04, Connector_JST:JST_PH_B4B-PH-K_1x04_P2.00mm_Vertical, symbol Connector_Generic:Conn_01x04
- added LS1: KLJ-1230, KLJ-1230_KKG, symbol 2026-10-16_01-37-39:KLJ-1230
- added SW1: CJS-1200B, CJS-1200B_NDC, symbol 2026-10-16_07-59-58:CJS-1200B
- added SW2: SW_Push, Button_Switch_THT:SW_PUSH_6mm, symbol Switch:SW_Push
Connections:
- net 2W_I2C_SCL: now also J23.4 (Pin_4)
- net 2W_I2C_SDA: now also J23.3 (Pin_3)
- net 3V3_AUX: now also J23.2 (Pin_2)
- net Buzzer: now also LS1.1
- net GND: now also D3.1 (K), D4.1 (K), D5.1 (K), D6.1 (K), J23.1 (Pin_1), LS1.2, SW1.2, SW2.1
- net LED1: now also D3.2 (A)
- net LED2: now also D4.2 (A)
- net SLIDER_2: now reaches J2.15 (Pin_15)
- net SLIDER_2: now also SW1.3
- net SLIDER_1: now reaches J2.16 (Pin_16)
- net SLIDER_1: now also SW1.1
- net SW_PUSH: now reaches J2.17 (Pin_17)
- net SW_PUSH: now also SW2.2
- net LED4: now reaches J2.19 (Pin_19)
- net LED4: now also D6.2 (A)
- net LED3: now reaches J2.20 (Pin_20)
- net LED3: now also D5.2 (A)
Other:
- note added: "UI"

Commit message: h
Parts:
- removed C22: 1000uF, Capacitor_SMD:CP_Elec_10x10.5, symbol Device:C_Polarized
Connections:
- net GND: now also C24.1
- no-connect marks 0 -> 10

Commit message: hj
Parts:
- J17: renamed from J10; footprint Connector_PinSocket_2.54mm:PinSocket_1x05_P2.54mm_Vertical -> Connector_JST:JST_PH_B5B-PH-K_1x05_P2.00mm_Vertical
- J19: renamed from J17; footprint Connector_JST:JST_PH_S3B-PH-K_1x03_P2.00mm_Horizontal -> Connector_JST:JST_PH_B3B-PH-K_1x03_P2.00mm_Vertical
- J20: renamed from J18; footprint Connector_JST:JST_PH_S3B-PH-K_1x03_P2.00mm_Horizontal -> Connector_JST:JST_PH_B3B-PH-K_1x03_P2.00mm_Vertical
- J21: renamed from J19; footprint Connector_JST:JST_PH_S3B-PH-K_1x03_P2.00mm_Horizontal -> Connector_JST:JST_PH_B3B-PH-K_1x03_P2.00mm_Vertical
- J22: renamed from J20; footprint Connector_JST:JST_PH_S3B-PH-K_1x03_P2.00mm_Horizontal -> Connector_JST:JST_PH_B3B-PH-K_1x03_P2.00mm_Vertical
- LS1: footprint KLJ-1230_KKG -> 独自:KLJ-1230_KKG-M; symbol 2026-10-16_01-37-39:KLJ-1230 -> 独自_sym:KLJ-1230
- SW2: renamed from SW1; footprint CJS-1200B_NDC -> 独自:CJS-1200B_NDC-M; symbol 2026-10-16_07-59-58:CJS-1200B -> 独自_sym:CJS-1200B
- U1, U2, U3, U4: footprint PWP0016J_N -> 独自:PWP0016J_N; symbol KiCADv6:DRV8874PWPR -> 独自_sym:DRV8874PWPR
- U8, U9: footprint IRLML6344TRPBF_INF -> 独自:IRLML6344TRPBF_INF-M; symbol 2026-10-05_00-38-08:IRLML6344TRPBF -> 独自_sym:IRLML6344TRPBF
- renumbered C5 to C1, C9 to C10, C14 to C11, C19 to C12, C1 to C13, C11 to C14, C16 to C15, C21 to C16, C4 to C17, C7 to C18, C12 to C19, C8 to C2, C17 to C20, C2 to C21, C24 to C22, C13 to C3, C18 to C4, C3 to C5, C10 to C6, C15 to C7, C20 to C8, C6 to C9, D3 to D1, D5 to D2, D4 to D3, D6 to D4, D1 to D5, D2 to D6, J23 to J1, J8 to J10, J3 to J11, J4 to J12, J1 to J13, J2 to J14, J12 to J15, J14 to J16, J9 to J18, J21 to J2, J22 to J3, J6 to J4, J7 to J6, J11 to J7, J13 to J8, J15 to J9, L2 to L1, L1 to L2, R2 to R1, R6 to R10, R9 to R11, R17 to R13, R16 to R14, R13 to R15, R14 to R16, R15 to R17, R4 to R2, R7 to R3, R10 to R4, R3 to R5, R5 to R6, R8 to R7, R11 to R8, R1 to R9, SW2 to SW1, TP3 to TP1, TP1 to TP2, TP2 to TP3, U1211 to U5, U121 to U6

Commit message: h
Parts:
- J1: footprint Connector_JST:JST_PH_B4B-PH-K_1x04_P2.00mm_Vertical -> EEDA:CONN-SMD_B4B-PH-SM4-TB-LF-SN
Changed lines of the file:
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@@
 			)
 		)
-		(property "Footprint" "Connector_JST:JST_PH_B4B-PH-K_1x04_P2.00mm_Vertical"
+		(property "Footprint" "EEDA:CONN-SMD_B4B-PH-SM4-TB-LF-SN"
 			(at 204.47 162.56 0)
 			(hide yes)
