File: PCB_Parts/main_board/main.kicad_sch (KiCad schematic)
At the start: 92 parts, among them J1 Conn_01x04, J10 Screw_Terminal_01x02, J11 Conn_01x20_Socket, J12 Conn_01x20_Socket, J13 Conn_01x20_Socket, J14 Conn_01x20_Socket, J15 Conn_01x04, J16 Conn_01x04, J17 Conn_01x05, J18 Screw_Terminal_01x02, J19 Conn_01x03, J2 Screw_Terminal_01x02, J20 Conn_01x03, J21 Conn_01x03, J22 Conn_01x03, J3 Screw_Terminal_01x02, J4 Screw_Terminal_01x02, J5 Conn_01x02, J6 Screw_Terminal_01x02, J7 Conn_01x04, J8 Conn_01x04, J9 Conn_01x08, SW1 SW_Push, SW2 CJS-1200B, U1 DRV8874PWPR, U2 DRV8874PWPR, U3 DRV8874PWPR, U4 DRV8874PWPR, U5 TPS62162DSG, U6 TPS62133, U7 ADS1015IDGS, U8 IRLML6344TRPBF, U9 IRLML6344TRPBF

Commit message: l
Parts:
- removed F1: 20A, Fuse:Fuse_1206_3216Metric, symbol Device:Fuse
- added C24, C28: 10nF, Capacitor_SMD:C_0603_1608Metric, symbol Device:C
- added C25: 100nF, Capacitor_SMD:C_0603_1608Metric, symbol Device:C
- added C26, C27: 22nF, Capacitor_SMD:C_0603_1608Metric, symbol Device:C
- added R19, R20, R21, R22: 470Ω, Resistor_SMD:R_0603_1608Metric, symbol Device:R
- J15, J16, J7, J8: footprint Connector_JST:JST_PH_B4B-PH-K_1x04_P2.00mm_Vertical -> EEDA:CONN-SMD_B4B-PH-SM4-TB-LF-SN
- J17: footprint Connector_JST:JST_PH_B5B-PH-K_1x05_P2.00mm_Vertical -> EEDA:CONN-SMD_5P-P2.00_B6B-PH-SM4-TB-LF-SN
- J19, J20, J21, J22: footprint Connector_JST:JST_PH_B3B-PH-K_1x03_P2.00mm_Vertical -> EEDA:CONN-SMD_B3B-PH-SM4-TB-LF-SN
- J9: footprint Connector_JST:JST_PH_B8B-PH-K_1x08_P2.00mm_Vertical -> EEDA:CONN-SMD_B8B-PH-SM4-TB-A
- TP1, TP2, TP3, TP4, TP5, TP6, TP7, TP8: footprint TestPoint:TestPoint_Plated_Hole_D2.0mm -> TestPoint:TestPoint_Pad_D3.0mm
Connections:
- net Pico_AGND is gone; now on net GND: J11.13 (Pin_13), J11.18 (Pin_18), J11.3 (Pin_3), J11.8 (Pin_8), J12.13 (Pin_13), J12.18 (Pin_18), J12.3 (Pin_3), J12.8 (Pin_8)
- net 2W_RUN: now also J14.11 (Pin_11); no longer J14.12 (Pin_12)
- net 3V3_AUX: now also C27.2
- net 5V: now also C26.2, C28.2; no longer U5.2 (VIN)
- net GND: now also J13.13 (Pin_13), J13.18 (Pin_18), J13.3 (Pin_3), J13.8 (Pin_8), J14.13 (Pin_13), J14.18 (Pin_18), J14.3 (Pin_3), J14.8 (Pin_8), C24.1, C25.1, C26.1, C27.1
- net LED1: now also R19.2; no longer D1.2 (A)
- net LED2: now also R20.1; no longer D3.2 (A)
- net LED3: now also R22.2; no longer D2.2 (A)
- net LED4: now also R21.1; no longer D4.2 (A)
- net VBAT_ADC: now also J14.10 (Pin_10); no longer J14.11 (Pin_11)
- net VBAT_FUSED: now also C23.1, J5.2 (Pin_2), C24.2, C25.2
- removed net 2W_AGND: J13.13 (Pin_13), J13.18 (Pin_18), J13.3 (Pin_3), J13.8 (Pin_8), J14.14 (Pin_14), J14.18 (Pin_18), J14.3 (Pin_3), J14.8 (Pin_8)
- new net: D1.2 (A), R19.1
- new net: C28.1, U5.2 (VIN)
- new net: D4.2 (A), R21.2
- new net: D3.2 (A), R20.2
- new net: D2.2 (A), R22.1

Commit message: h
Parts:
- C24, C28: value 10nF -> 10uF
- C26, C27: value 22nF -> 22uF
Connections:
- net 5V: now also U5.2 (VIN)
- net GND: now also C28.1
Other:
- moved on the sheet: C28
Changed lines of the file:
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@@
 	)
 	(label "5V"
-		(at 119.38 118.11 180)
+		(at 127 118.11 180)
 		(effects
 			(font
@@
 			)
 		)
-		(property "Value" "10nF"
+		(property "Value" "10uF"
 			(at 86.36 109.22 90)
 			(show_name no)
@@
 			)
 		)
-		(property "Value" "22nF"
+		(property "Value" "22uF"
 			(at 158.75 123.1899 0)
 			(show_name no)
@@
 	(symbol
 		(lib_id "Device:C")
-		(at 123.19 118.11 270)
+		(at 127 114.3 0)
 		(unit 1)
 		(body_style 1)
@@
 		(fields_autoplaced yes)
 		(property "Reference" "C28"
-			(at 123.19 110.49 90)
+			(at 130.81 113.0299 0)
 			(show_name no)
 			(do_not_autoplace no)
@@
 					(size 1.27 1.27)
 				)
+				(justify left)
 			)
 		)
-		(property "Value" "10nF"
-			(at 123.19 113.03 90)
+		(property "Value" "10uF"
+			(at 130.81 115.5699 0)
 			(show_name no)
 			(do_not_autoplace no)
@@
 					(size 1.27 1.27)
 				)
+				(justify left)
 			)
 		)
 		(property "Footprint" "Capacitor_SMD:C_0603_1608Metric"
-			(at 119.38 119.0752 0)
+			(at 127.9652 118.11 0)
 			(hide yes)
 			(show_name no)
@@
 		)
 		(property "Datasheet" ""
-			(at 123.19 118.11 0)
+			(at 127 114.3 0)
 			(hide yes)
 			(show_name no)
@@
 		)
 		(property "Description" "Unpolarized capacitor"
-			(at 123.19 118.11 0)
+			(at 127 114.3 0)
 			(hide yes)
 			(show_name no)
@@
 	)
 	(symbol
+		(lib_id "power:GND")
+		(at 127 110.49 90)
+		(unit 1)
+		(body_style 1)
+		(exclude_from_sim no)
+		(in_bom yes)
+		(on_board yes)
+		(in_pos_files yes)
+		(dnp no)
+		(fields_autoplaced yes)
+		(property "Reference" "#PWR097"
+			(at 133.35 110.49 0)
+			(hide yes)
+			(show_name no)
+			(do_not_autoplace no)
+			(effects
+				(font
+					(size 1.27 1.27)
+				)
+			)
+		)
+		(property "Value" "GND"
+			(at 130.81 110.4899 90)
+			(show_name no)
+			(do_not_autoplace no)
+			(effects
+				(font
+					(size 1.27 1.27)
+				)
+				(justify right)
+			)
+		)
+		(property "Footprint" ""
+			(at 127 110.49 0)
+			(hide yes)
+			(show_name no)
+			(do_not_autoplace no)
+			(effects
+				(font
+					(size 1.27 1.27)
+				)
+			)
+		)
+		(property "Datasheet" ""
+			(at 127 110.49 0)
+			(hide yes)
+			(show_name no)
+			(do_not_autoplace no)
+			(effects
+				(font
+					(size 1.27 1.27)
+				)
+			)
+		)
+		(property "Description" "Power symbol creates a global label with name \"GND\" , ground"
+			(at 127 110.49 0)
+			(hide yes)
+			(show_name no)
+			(do_not_autoplace no)
+			(effects
+				(font
+					(size 1.27 1.27)
+				)
+			)
+		)
+		(pin "1"
+		)
+		(instances
+			(project "main"
+				(path "/2092c9bc-9fbe-439d-a80c-904a7787fec4"
+					(reference "#PWR097")
+					(unit 1)
+				)
+			)
+		)
+	)
+	(symbol
 		(lib_id "Device:C")
 		(at 83.82 69.85 0)
@@
 			)
 		)
-		(property "Value" "22nF"
+		(property "Value" "22uF"
 			(at 111.76 126.9999 0)
 			(show_name no)
