File: PCB_Parts/main_board/main.kicad_pcb (KiCad board)
At the start: 2 copper layers, 92 parts, among them J1 Conn_01x04, J10 Screw_Terminal_01x02, J11 Conn_01x20_Socket, J12 Conn_01x20_Socket, J13 Conn_01x20_Socket, J14 Conn_01x20_Socket, J15 Conn_01x04, J16 Conn_01x04, J17 Conn_01x05, J18 Screw_Terminal_01x02, J19 Conn_01x03, J2 Screw_Terminal_01x02, J20 Conn_01x03, J21 Conn_01x03, J22 Conn_01x03, J3 Screw_Terminal_01x02, J4 Screw_Terminal_01x02, J5 Conn_01x02, J6 Screw_Terminal_01x02, J7 Conn_01x04, J8 Conn_01x04, J9 Conn_01x08, SW1 SW_Push, SW2 CJS-1200B, U1 DRV8874PWPR, U2 DRV8874PWPR, U3 DRV8874PWPR, U4 DRV8874PWPR, U5 TPS62162DSG, U6 TPS62133, U7 ADS1015IDGS, U8 IRLML6344TRPBF, U9 IRLML6344TRPBF

Commit message: f
Parts:
- moved U8 119.0 mm to (43.5, 60.5), turned to 90 degrees
- moved U9 117.9 mm to (43.5, 73.0), turned to 90 degrees
- moved J11 101.5 mm to (77.6, 156.5)
- moved J12 101.5 mm to (82.2, 156.5)
- moved J13 101.5 mm to (86.8, 156.5)
- moved J14 101.5 mm to (91.3, 156.5)
- moved U4 96.1 mm to (43.0, 120.8), turned to -90 degrees
- moved U3 93.5 mm to (43.2, 108.5), turned to -90 degrees
- moved U2 91.1 mm to (43.5, 96.0), turned to -90 degrees
- moved U1 89.5 mm to (43.5, 84.5), turned to -90 degrees
- moved R15 86.3 mm to (49.0, 60.5)
- moved R14 85.4 mm to (49.0, 73.0)
- moved R16 82.9 mm to (53.5, 60.5)
- moved D5 82.8 mm to (65.0, 60.0)
- moved D6 82.4 mm to (65.0, 72.5)
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
Commit message: h
Parts:
- J1, J15, J16, J7, J8: footprint Connector_JST:JST_PH_B4B-PH-K_1x04_P2.00mm_Vertical -> EEDA:CONN-SMD_B4B-PH-SM4-TB-LF-SN
- J17: footprint Connector_JST:JST_PH_B5B-PH-K_1x05_P2.00mm_Vertical -> EEDA:CONN-SMD_5P-P2.00_B6B-PH-SM4-TB-LF-SN
- J19, J20, J21, J22: footprint Connector_JST:JST_PH_B3B-PH-K_1x03_P2.00mm_Vertical -> EEDA:CONN-SMD_B3B-PH-SM4-TB-LF-SN
- J9: footprint Connector_JST:JST_PH_B8B-PH-K_1x08_P2.00mm_Vertical -> EEDA:CONN-SMD_B8B-PH-SM4-TB-A
- moved J5 111.8 mm to (41.3, 133.4), turned to 90 degrees
- moved J14 103.8 mm to (119.4, 56.5)
- moved J13 101.1 mm to (101.6, 56.5)
- moved J11 100.4 mm to (68.6, 56.5)
- moved J12 100.1 mm to (86.4, 56.5)
- moved F1 96.5 mm to (60.8, 141.6)
- moved C23 93.3 mm to (50.8, 136.2), turned to 90 degrees
- moved L2 91.4 mm to (54.8, 63.5), turned to 90 degrees
- moved L1 86.4 mm to (59.7, 56.6)
- moved D1 85.9 mm to (139.2, 57.8), turned to 180 degrees
- moved D2 85.9 mm to (139.2, 61.2), turned to 180 degrees
- moved D4 85.9 mm to (139.2, 67.9), turned to 180 degrees
- moved D3 85.9 mm to (139.2, 64.6), turned to 180 degrees
- moved U5 84.5 mm to (55.7, 56.7)
- moved J1 76.9 mm to (126.4, 133.3), turned to 180 degrees
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Other:
- board text added: "BNO085"
- board text added: "IR"
- board text added: "Line"
- board text added: "Pico"
- board text added: "Pico2W"
- board text added: "SuperSonic"

Commit message: haisen
Parts:
- moved TP5 95.5 mm to (50.8, 55.2)
- moved TP4 83.8 mm to (51.4, 72.4)
- moved TP1 82.9 mm to (58.4, 55.2)
- moved TP3 78.1 mm to (55.2, 72.4)
- moved TP6 66.6 mm to (64.8, 92.1)
- moved TP7 66.3 mm to (67.3, 135.9)
- moved TP2 57.7 mm to (61.0, 135.9)
- moved TP8 36.9 mm to (128.9, 82.5)
- moved R12 10.8 mm to (56.7, 121.3), turned to 180 degrees
- moved R4 10.5 mm to (51.9, 118.1), turned to 180 degrees
- moved C21 9.06 mm to (59.9, 72.1), turned to 90 degrees
- moved C20 8.85 mm to (47.5, 118.1), turned to 180 degrees
- moved C8 8.51 mm to (47.5, 123.8), turned to 180 degrees
- moved R8 7.78 mm to (56.7, 118.1), turned to 0 degrees
- moved C16 7.30 mm to (52.1, 121.3), turned to 0 degrees
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Routing:
- net GND: track 0.00 -> 188.6 mm, vias 0 -> 84
- net /RIGHT_TRIG: track 0.00 -> 137.0 mm, vias 0 -> 2
- net /2W_I2C_SDA: track 0.00 -> 126.1 mm, vias 0 -> 10
- net /2W_I2C_SCL: track 0.00 -> 119.9 mm, vias 0 -> 8
- net /REAR_ECHO: track 0.00 -> 116.9 mm, vias 0 -> 2
- net /Pico_AGND: track 0.00 -> 114.4 mm, vias 0 -> 7
- net /LEFT_TRIG: track 0.00 -> 110.4 mm, vias 0 -> 2
- net /2W_AGND: track 0.00 -> 105.2 mm, vias 0 -> 5
- net /DRV_nFAULT: track 0.00 -> 102.6 mm, vias 0 -> 7
- net /LEFT_ECHO: track 0.00 -> 99.9 mm, vias 0 -> 2
- net /DRV_nSLEEP: track 0.00 -> 96.9 mm, vias 0 -> 8
- net /RIGHT_ECHO: track 0.00 -> 90.4 mm, vias 0 -> 6
- net /FRONT_TRIG: track 0.00 -> 83.7 mm, vias 0 -> 6
- net /FRONT_ECHO: track 0.00 -> 82.9 mm, vias 0 -> 6
- net /REAR_TRIG: track 0.00 -> 79.9 mm, vias 0 -> 6
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- added copper zone on B.Cu, net GND
Other:
- board outline added: 138.4 x 94 mm

Commit message: aaa
Connections:
- U5 pad 6: /3V3_AUX -> Net-(U5-SW)
Routing:
- net GND: track 188.6 -> 226.9 mm, vias 84 -> 85
- net /DRIB_MOTOR_SW: track 0.00 -> 32.1 mm
- net Net-(J5-Pin_2): track 0.00 -> 29.6 mm, vias 0 -> 3
- net /VBAT_FUSED: track 0.00 -> 24.0 mm
- net /3V3_AUX: track 0.00 -> 5.84 mm
- net Net-(U5-SW): track 0.00 -> 2.40 mm
Changed lines of the file:
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@@
 			(layers "F.Cu" "F.Mask" "F.Paste")
 			(roundrect_rratio 0.25)
-			(net "/3V3_AUX")
+			(net "Net-(U5-SW)")
 			(pinfunction "VOS_6")
 			(pintype "input")
@@
 	)
 	(segment
+		(start 49.385 133.43)
+		(end 50.84 131.975)
+		(width 2.5)
+		(layer "F.Cu")
+		(net "GND")
+	)
+	(segment
 		(start 46.2 109.2)
 		(end 46.2 108.8)
@@
 	)
 	(segment
+		(start 67.31 135.89)
+		(end 63.395 131.975)
+		(width 3)
+		(layer "F.Cu")
+		(net "GND")
+	)
+	(segment
 		(start 140.6 57.8)
 		(end 140.595 57.775)
@@
 	)
 	(segment
+		(start 63.395 131.975)
+		(end 50.84 131.975)
+		(width 3)
+		(layer "F.Cu")
+		(net "GND")
+	)
+	(segment
 		(start 40.284999 105.524601)
 		(end 40.3 105.5)
@@
 	)
 	(segment
+		(start 41.275 133.43)
+		(end 49.385 133.43)
+		(width 2.5)
+		(layer "F.Cu")
+		(net "GND")
+	)
+	(segment
 		(start 108.2 117.8)
 		(end 107.2 116.8)
@@
 	)
 	(via
+		(at 50.84 131.975)
+		(size 0.6)
+		(drill 0.3)
+		(layers "F.Cu" "B.Cu")
+		(net "GND")
+	)
+	(via
 		(at 47 105.5)
 		(size 0.6)
@@
 	)
 	(segment
+		(start 41.275 133.43)
+		(end 49.37 133.43)
+		(width 2.5)
+		(layer "B.Cu")
+		(net "GND")
+	)
+	(segment
 		(start 125.3 85.72)
 		(end 125.3 85.7)
@@
 	)
 	(segment
+		(start 49.37 133.43)
+		(end 50.8 132)
+		(width 2.5)
+		(layer "B.Cu")
+		(net "GND")
+	)
+	(segment
 		(start 125.25 82.57)
 		(end 125.2 82.6)
@@
 	)
 	(segment
+		(start 58.42 55.245)
+		(end 58.42 59.9425)
+		(width 0.5)
+		(layer "F.Cu")
+		(net "/3V3_AUX")
+	)
+	(segment
+		(start 58.42 59.9425)
+		(end 59.2275 60.75)
+		(width 0.5)
+		(layer "F.Cu")
+		(net "/3V3_AUX")
+	)
+	(segment
 		(start 126.6 101.1)
 		(end 136.6 111.1)
@@
 	)
 	(segment
+		(start 45.72 53.82)
+		(end 45.72 57.055)
+		(width 2.5)
+		(layer "F.Cu")
+		(net "/VBAT_FUSED")
+	)
+	(segment
+		(start 36.965 53.82)
+		(end 45.72 53.82)
+		(width 2.5)
+		(layer "F.Cu")
+		(net "/VBAT_FUSED")
+	)
+	(segment
+		(start 33 57.785)
+		(end 36.965 53.82)
+		(width 2.5)
+		(layer "F.Cu")
+		(net "/VBAT_FUSED")
+	)
+	(segment
+		(start 45.72 57.055)
+		(end 45.815 57.15)
+		(width 2.5)
+		(layer "F.Cu")
+		(net "/VBAT_FUSED")
+	)
+	(segment
+		(start 62.23 137.16)
+		(end 60.96 135.89)
+		(width 1)
+		(layer "F.Cu")
+		(net "/VBAT_FUSED")
+	)
+	(segment
+		(start 62.23 141.605)
+		(end 62.23 137.16)
+		(width 1)
+		(layer "F.Cu")
+		(net "/VBAT_FUSED")
+	)
+	(segment
 		(start 44.8 75.5)
 		(end 44.8 74.5)
@@
 	)
 	(segment
+		(start 55.0225 60.6)
+		(end 56.7075 60.6)
+		(width 0.3)
+		(layer "F.Cu")
+		(net "Net-(U5-SW)")
+	)
+	(segment
+		(start 55.0225 61.1)
+		(end 55.0225 60.6)
+		(width 0.3)
+		(layer "F.Cu")
+		(net "Net-(U5-SW)")
+	)
+	(segment
+		(start 56.7075 60.6)
+		(end 56.8575 60.75)
+		(width 0.3)
+		(layer "F.Cu")
+		(net "Net-(U5-SW)")
+	)
+	(segment
 		(start 40.9 93.6)
 		(end 40.934998 93.570001)
@@
 	)
 	(segment
+		(start 46.355 59.69)
+		(end 36.175 59.69)
+		(width 0.5)
+		(layer "F.Cu")
+		(net "/DRIB_MOTOR_SW")
+	)
+	(segment
+		(start 38.715 57.15)
+		(end 33 62.865)
+		(width 2.5)
+		(layer "F.Cu")
+		(net "/DRIB_MOTOR_SW")
+	)
+	(segment
+		(start 36.175 59.69)
+		(end 33 62.865)
+		(width 0.5)
+		(layer "F.Cu")
+		(net "/DRIB_MOTOR_SW")
+	)
+	(segment
+		(start 41.815 57.15)
+		(end 38.715 57.15)
+		(width 2.5)
+		(layer "F.Cu")
+		(net "/DRIB_MOTOR_SW")
+	)
+	(segment
+		(start 50.8 55.245)
+		(end 46.355 59.69)
+		(width 0.5)
+		(layer "F.Cu")
+		(net "/DRIB_MOTOR_SW")
+	)
+	(segment
+		(start 48.895 138.43)
+		(end 50.84 140.375)
+		(width 5)
+		(layer "F.Cu")
+		(net "Net-(J5-Pin_2)")
+	)
+	(segment
+		(start 59.43 141.605)
+		(end 53.975 141.605)
+		(width 3)
+		(layer "F.Cu")
+		(net "Net-(J5-Pin_2)")
+	)
+	(segment
+		(start 52.07 141.605)
+		(end 53.975 141.605)
+		(width 3)
+		(layer "F.Cu")
+		(net "Net-(J5-Pin_2)")
+	)
+	(segment
+		(start 50.84 140.375)
+		(end 52.07 141.605)
+		(width 3)
+		(layer "F.Cu")
+		(net "Net-(J5-Pin_2)")
+	)
+	(segment
+		(start 41.275 138.43)
+		(end 48.895 138.43)
+		(width 5)
+		(layer "F.Cu")
+		(net "Net-(J5-Pin_2)")
+	)
+	(via
+		(at 57.15 141.605)
+		(size 0.6)
+		(drill 0.3)
+		(layers "F.Cu" "B.Cu")
+		(net "Net-(J5-Pin_2)")
+	)
+	(via
+		(at 48.895 138.43)
+		(size 0.6)
+		(drill 0.3)
+		(layers "F.Cu" "B.Cu")
+		(net "Net-(J5-Pin_2)")
+	)
+	(via
+		(at 53.975 141.605)
+		(size 0.6)
+		(drill 0.3)
+		(layers "F.Cu" "B.Cu")
+		(net "Net-(J5-Pin_2)")
+	)
+	(segment
+		(start 41.275 138.43)
+		(end 48.895 138.43)
+		(width 5)
+		(layer "B.Cu")
+		(net "Net-(J5-Pin_2)")
+	)
+	(segment
+		(start 53.975 141.605)
+		(end 56.515 141.605)
+		(width 3)
+		(layer "B.Cu")
+		(net "Net-(J5-Pin_2)")
+	)
+	(segment

Commit message: 2
Routing:
- net /VBAT_ADC: track 0.00 -> 23.7 mm, vias 0 -> 3
- net /VBAT_FUSED: track 24.0 -> 37.9 mm
- net /KICK_SW: track 0.00 -> 11.1 mm
Changed lines of the file:
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@@
 	)
 	(segment
-		(start 45.72 53.82)
-		(end 45.72 57.055)
-		(width 2.5)
+		(start 36.83 66.04)
+		(end 33 69.87)
+		(width 2)
 		(layer "F.Cu")
 		(net "/VBAT_FUSED")
 	)
 	(segment
-		(start 36.965 53.82)
-		(end 45.72 53.82)
-		(width 2.5)
+		(start 36.81 53.975)
+		(end 33 57.785)
+		(width 2)
 		(layer "F.Cu")
 		(net "/VBAT_FUSED")
 	)
 	(segment
-		(start 33 57.785)
-		(end 36.965 53.82)
-		(width 2.5)
+		(start 45.72 69.215)
+		(end 42.545 66.04)
+		(width 2)
 		(layer "F.Cu")
 		(net "/VBAT_FUSED")
 	)
 	(segment
-		(start 45.72 57.055)
-		(end 45.815 57.15)
-		(width 2.5)
+		(start 45.815 56.61)
+		(end 43.18 53.975)
+		(width 2)
+		(layer "F.Cu")
+		(net "/VBAT_FUSED")
+	)
+	(segment
+		(start 33 69.87)
+		(end 33 69.91)
+		(width 2)
+		(layer "F.Cu")
+		(net "/VBAT_FUSED")
+	)
+	(segment
+		(start 42.545 66.04)
+		(end 36.83 66.04)
+		(width 2)
 		(layer "F.Cu")
 		(net "/VBAT_FUSED")
@@
 	)
 	(segment
+		(start 45.815 57.15)
+		(end 45.815 56.61)
+		(width 2)
+		(layer "F.Cu")
+		(net "/VBAT_FUSED")
+	)
+	(segment
 		(start 62.23 141.605)
 		(end 62.23 137.16)
@@
 	)
 	(segment
+		(start 43.18 53.975)
+		(end 36.81 53.975)
+		(width 2)
+		(layer "F.Cu")
+		(net "/VBAT_FUSED")
+	)
+	(segment
+		(start 123.685 83.325)
+		(end 123.685 82.55)
+		(width 0.2)
+		(layer "F.Cu")
+		(net "/VBAT_ADC")
+	)
+	(segment
+		(start 122.122646 84.022646)
+		(end 122.987354 84.022646)
+		(width 0.2)
+		(layer "F.Cu")
+		(net "/VBAT_ADC")
+	)
+	(segment
+		(start 123.635 85.725)
+		(end 122.122646 84.212646)
+		(width 0.2)
+		(layer "F.Cu")
+		(net "/VBAT_ADC")
+	)
+	(segment
+		(start 122.555 79.375)
+		(end 121.92 80.01)
+		(width 0.2)
+		(layer "F.Cu")
+		(net "/VBAT_ADC")
+	)
+	(segment
+		(start 119.38 81.915)
+		(end 120.65 83.185)
+		(width 0.2)
+		(layer "F.Cu")
+		(net "/VBAT_ADC")
+	)
+	(segment
+		(start 123.635 79.375)
+		(end 122.555 79.375)
+		(width 0.2)
+		(layer "F.Cu")
+		(net "/VBAT_ADC")
+	)
+	(segment
+		(start 120.65 83.185)
+		(end 121.285 83.185)
+		(width 0.2)
+		(layer "F.Cu")
+		(net "/VBAT_ADC")
+	)
+	(segment
+		(start 122.122646 84.212646)
+		(end 122.122646 84.022646)
+		(width 0.2)
+		(layer "F.Cu")
+		(net "/VBAT_ADC")
+	)
+	(segment
+		(start 122.987354 84.022646)
+		(end 123.685 83.325)
+		(width 0.2)
+		(layer "F.Cu")
+		(net "/VBAT_ADC")
+	)
+	(via
+		(at 122.122646 84.022646)
+		(size 0.6)
+		(drill 0.3)
+		(layers "F.Cu" "B.Cu")
+		(net "/VBAT_ADC")
+	)
+	(via
+		(at 121.285 83.185)
+		(size 0.6)
+		(drill 0.3)
+		(layers "F.Cu" "B.Cu")
+		(net "/VBAT_ADC")
+	)
+	(via
+		(at 121.92 80.01)
+		(size 0.6)
+		(drill 0.3)
+		(layers "F.Cu" "B.Cu")
+		(net "/VBAT_ADC")
+	)
+	(segment
+		(start 121.92 80.01)
+		(end 121.285 80.645)
+		(width 0.2)
+		(layer "B.Cu")
+		(net "/VBAT_ADC")
+	)
+	(segment
+		(start 121.285 80.645)
+		(end 120.65 80.645)
+		(width 0.2)
+		(layer "B.Cu")
+		(net "/VBAT_ADC")
+	)
+	(segment
+		(start 121.285 83.185)
+		(end 122.122646 84.022646)
+		(width 0.2)
+		(layer "B.Cu")
+		(net "/VBAT_ADC")
+	)
+	(segment
+		(start 125.73 81.915)
+		(end 126.365 82.55)
+		(width 0.2)
+		(layer "B.Cu")
+		(net "/VBAT_ADC")
+	)
+	(segment
+		(start 120.65 80.645)
+		(end 119.38 81.915)
+		(width 0.2)
+		(layer "B.Cu")
+		(net "/VBAT_ADC")
+	)
+	(segment
+		(start 119.38 81.915)
+		(end 125.73 81.915)
+		(width 0.2)
+		(layer "B.Cu")
+		(net "/VBAT_ADC")
+	)
+	(segment
+		(start 126.365 82.55)
+		(end 128.905 82.55)
+		(width 0.2)
+		(layer "B.Cu")
+		(net "/VBAT_ADC")
+	)
+	(segment
 		(start 44.8 75.5)
 		(end 44.8 74.5)
@@
 	)
 	(segment
+		(start 35.5 74.99)
+		(end 33 74.99)
+		(width 2)
+		(layer "F.Cu")
+		(net "/KICK_SW")
+	)
+	(segment
+		(start 41.72 69.215)
+		(end 41.275 69.215)
+		(width 2)
+		(layer "F.Cu")
+		(net "/KICK_SW")
+	)
+	(segment
+		(start 41.275 69.215)
+		(end 35.5 74.99)
+		(width 2)
+		(layer "F.Cu")
+		(net "/KICK_SW")
+	)
+	(segment
 		(start 41.2 80.5)
 		(end 41.199999 81.524601)
@@
 	)
 	(segment
-		(start 38.715 57.15)
-		(end 33 62.865)
-		(width 2.5)
+		(start 41.815 57.15)
+		(end 38.715 57.15)
+		(width 2)
 		(layer "F.Cu")
 		(net "/DRIB_MOTOR_SW")
@@
 	)
 	(segment
-		(start 41.815 57.15)
-		(end 38.715 57.15)
-		(width 2.5)
+		(start 38.715 57.15)
+		(end 33 62.865)
+		(width 2)
 		(layer "F.Cu")
 		(net "/DRIB_MOTOR_SW")

Commit message: l
Parts:
- removed F1: 20A, Fuse:Fuse_1206_3216Metric
- added C24: 10nF, Capacitor_SMD:C_0603_1608Metric, F.Cu at (58.2, 72.1)
- added C25: 100nF, Capacitor_SMD:C_0603_1608Metric, F.Cu at (63.7, 64.1)
- added C26: 22nF, Capacitor_SMD:C_0603_1608Metric, F.Cu at (49.2, 66.5)
- added C27: 22nF, Capacitor_SMD:C_0603_1608Metric, F.Cu at (61.8, 58.2)
- added C28: 10nF, Capacitor_SMD:C_0603_1608Metric, F.Cu at (50.8, 61.9)
- added R19: 470Ω, Resistor_SMD:R_0603_1608Metric, F.Cu at (144.9, 60.6)
- added R20: 470Ω, Resistor_SMD:R_0603_1608Metric, F.Cu at (145.0, 65.5)
- added R21: 470Ω, Resistor_SMD:R_0603_1608Metric, F.Cu at (145.0, 68.0)
- added R22: 470Ω, Resistor_SMD:R_0603_1608Metric, F.Cu at (145.0, 62.9)
- TP1, TP2, TP3, TP4, TP5, TP6, TP7, TP8: footprint TestPoint:TestPoint_Plated_Hole_D2.0mm -> TestPoint:TestPoint_Pad_D3.0mm
- moved C9 12.0 mm to (40.5, 90.6)
- moved C10 11.8 mm to (40.6, 102.5)
- moved D1 11.5 mm to (150.4, 60.3)
- moved D2 11.3 mm to (150.4, 62.9)
- moved D3 11.2 mm to (150.4, 65.4)
- moved D4 11.2 mm to (150.4, 67.9)
- moved TP6 11.1 mm to (72.6, 99.9)
- moved C12 10.6 mm to (41.9, 127.4)
- moved C11 10.3 mm to (42.1, 114.3)
- moved TP3 0.11 mm to (55.3, 72.4)
Connections:
- C23 pad 1: Net-(J5-Pin_2) -> /VBAT_FUSED
- D1 pad 2: /LED1 -> Net-(D1-A)
- D2 pad 2: /LED3 -> Net-(D2-A)
- D3 pad 2: /LED2 -> Net-(D3-A)
- D4 pad 2: /LED4 -> Net-(D4-A)
- J11 pad 13: /Pico_AGND -> GND
- J11 pad 18: /Pico_AGND -> GND
- J11 pad 3: /Pico_AGND -> GND
- J11 pad 8: /Pico_AGND -> GND
- J12 pad 13: /Pico_AGND -> GND
- J12 pad 18: /Pico_AGND -> GND
- J12 pad 3: /Pico_AGND -> GND
- J12 pad 8: /Pico_AGND -> GND
- J13 pad 13: /2W_AGND -> GND
- J13 pad 18: /2W_AGND -> GND
- J13 pad 3: /2W_AGND -> GND
- J13 pad 8: /2W_AGND -> GND
- J14 pad 10: unconnected-(J14-Pin_10-Pad10) -> /VBAT_ADC
- J14 pad 11: /VBAT_ADC -> /2W_RUN
- J14 pad 12: /2W_RUN -> unconnected-(J14-Pin_12-Pad12)
- J14 pad 13: unconnected-(J14-Pin_13-Pad13) -> GND
- J14 pad 14: /2W_AGND -> unconnected-(J14-Pin_14-Pad14)
- J14 pad 18: /2W_AGND -> GND
- J14 pad 3: /2W_AGND -> GND
- J14 pad 8: /2W_AGND -> GND
- J5 pad 2: Net-(J5-Pin_2) -> /VBAT_FUSED
- U5 pad 2: /5V -> Net-(U5-VIN)
- U5 pad 6: Net-(U5-SW) -> /3V3_AUX
Routing:
- net /VBAT_FUSED: track 37.9 -> 515.9 mm, vias 0 -> 35
- net /3V3_AUX: track 5.84 -> 459.3 mm, vias 0 -> 18
- net /Pico_AGND: track 114.4 -> 0.00 mm, vias 7 -> 0
- net /2W_AGND: track 105.2 -> 0.00 mm, vias 5 -> 0
- net /5V: track 0.00 -> 99.5 mm, vias 0 -> 7
- net GND: track 226.9 -> 193.9 mm, vias 85 -> 94
- net Net-(J5-Pin_2): track 29.6 -> 0.00 mm, vias 3 -> 0
- net /KICK_SW: track 11.1 -> 38.4 mm, vias 0 -> 2
- net /DRIB_MOTOR_SW: track 32.1 -> 59.3 mm
- net /LEFT_TRIG: track 110.4 -> 137.5 mm
- net /LEFT_ECHO: track 99.9 -> 126.4 mm
- net /DRV_nSLEEP: track 96.9 -> 110.6 mm, vias 8 -> 11
- net /DRV_nFAULT: track 102.6 -> 116.0 mm, vias 7 -> 16
- net /REAR_ECHO: track 116.9 -> 130.1 mm
- net /RIGHT_TRIG: track 137.0 -> 148.9 mm
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- added copper zone on F.Cu, net /MOTOR1_OUT1
- added copper zone on F.Cu, net /MOTOR1_OUT2
- added copper zone on F.Cu, net /MOTOR2_OUT1
- added copper zone on F.Cu, net /MOTOR2_OUT2
- added copper zone on F.Cu, net /MOTOR3_OUT1
- added copper zone on F.Cu, net /MOTOR3_OUT2
- added copper zone on F.Cu, net /MOTOR4_OUT1
- added copper zone on F.Cu, net /MOTOR4_OUT2
- added copper zone on B.Cu, net /VBAT_FUSED
- added copper zone on F.Cu, net /VBAT_FUSED
- added copper zone on F.Cu, net GND
Other:
- board size 138.4 x 94 mm -> 138.4 x 100.9 mm

Commit message: h
Parts:
- C24, C28: value 10nF -> 10uF
- C26, C27: value 22nF -> 22uF
- moved TP4 0.21 mm to (51.2, 72.3)
Connections:
- C28 pad 1: Net-(U5-VIN) -> GND
- U5 pad 2: Net-(U5-VIN) -> /5V
Routing:
- net /5V: track 99.5 -> 105.2 mm, vias 7 -> 9
- net /DRV_nFAULT: track 116.0 -> 120.0 mm
- net /2W_I2C_SDA: track 126.1 -> 130.0 mm
- net Net-(U5-VIN): track 3.72 -> 0.00 mm
- net /2W_I2C_SCL: track 123.8 -> 127.4 mm
- net GND: track 193.9 -> 195.6 mm, vias 94 -> 93
