File: PCB_Parts/IR_sensor_ring/IR_sensor_ring.kicad_sch (KiCad schematic)
At the start: 0 parts

Commit message: irring
Parts:
- added C1, C10, C11, C12, C13, C14, C15, C16, C2, C3, C4, C5, C6, C7, C8, C9: 2.2nF, Capacitor_SMD:C_0603_1608Metric, symbol Device:C
- added J1: Conn_01x10, EEDA:CONN-SMD_B10B-PH-SM4-TB-LF-SN, symbol Connector_Generic:Conn_01x10
- added R1, R10, R11, R12, R13, R14, R15, R16, R2, R3, R4, R5, R6, R7, R8, R9: 47kΩ, Resistor_SMD:R_0508_1220Metric, symbol Device:R
- added U1, U10, U11, U12, U13, U14, U15, U16, U2, U3, U4, U5, U6, U7, U8, U9: VEMD10940FX01, EEDA:LED-SMD_3P-L3.0-W2.0_LTE-S3201L-ZB-HT, symbol Device:D_Photo
Connections:
- new net 3v3: U1.1 (K), U10.1 (K), U11.1 (K), U12.1 (K), U13.1 (K), U14.1 (K), U15.1 (K), U16.1 (K), U2.1 (K), U3.1 (K), U4.1 (K), U5.1 (K), U6.1 (K), U7.1 (K), U8.1 (K), U9.1 (K)
- new net GND: C1.1, C10.1, C11.1, C12.1, C13.1, C14.1, C15.1, C16.1, C2.1, C3.1, C4.1, C5.1, C6.1, C7.1, C8.1, C9.1, R1.2, R10.2, R11.2, R12.2, R13.2, R14.2, R15.2, R16.2, R2.2, R3.2, R4.2, R5.2, R6.2, R7.2, R8.2, R9.2
- new net IR1: C1.2, R1.1, U1.2 (A)
- new net IR10: C10.2, R10.1, U10.2 (A)
- new net IR11: C11.2, R11.1, U11.2 (A)
- new net IR12: C12.2, R12.1, U12.2 (A)
- new net IR13: C13.2, R13.1, U13.2 (A)
- new net IR14: C14.2, R14.1, U14.2 (A)
- new net IR15: C15.2, R15.1, U15.2 (A)
- new net IR16: C16.2, R16.1, U16.2 (A)
- new net IR2: C2.2, R2.1, U2.2 (A)
- new net IR3: C3.2, R3.1, U3.2 (A)
- new net IR4: C4.2, R4.1, U4.2 (A)
- new net IR5: C5.2, R5.1, U5.2 (A)
- new net IR6: C6.2, R6.1, U6.2 (A)
- new net IR7: C7.2, R7.1, U7.2 (A)
- new net IR8: C8.2, R8.1, U8.2 (A)
- new net IR9: C9.2, R9.1, U9.2 (A)

Commit message: IRRING CMP
Parts:
- added J2: Conn_01x10, EEDA:CONN-SMD_B10B-PH-SM4-TB-LF-SN, symbol Connector_Generic:Conn_01x10
- R1, R10, R11, R12, R13, R14, R15, R16, R2, R3, R4, R5, R6, R7, R8, R9: footprint Resistor_SMD:R_0508_1220Metric -> Resistor_SMD:R_0603_1608Metric
Connections:
- net 3v3: now also J1.2 (Pin_2), J2.2 (Pin_2)
- net GND: now also J1.1 (Pin_1), J2.1 (Pin_1)
- net IR1: now also J1.10 (Pin_10)
- net IR10: now also J2.9 (Pin_9)
- net IR11: now also J2.8 (Pin_8)
- net IR12: now also J2.7 (Pin_7)
- net IR13: now also J2.6 (Pin_6)
- net IR14: now also J2.5 (Pin_5)
- net IR15: now also J2.4 (Pin_4)
- net IR16: now also J2.3 (Pin_3)
- net IR2: now also J1.9 (Pin_9)
- net IR3: now also J1.8 (Pin_8)
- net IR4: now also J1.7 (Pin_7)
- net IR5: now also J1.6 (Pin_6)
- net IR6: now also J1.5 (Pin_5)
- net IR7: now also J1.4 (Pin_4)
- net IR8: now also J1.3 (Pin_3)
- net IR9: now also J2.10 (Pin_10)
